Commit message: Same as last comit
The rest of the files

File: urdf/scara1.xacro (robot description, xacro)
@@ -1,4 +1,4 @@
 <?xml version="1.0" encoding="utf-8"?>
-<robot name="billy_v2" xmlns:xacro="http://www.ros.org/wiki/xacro">
+<robot name="scara1" xmlns:xacro="http://www.ros.org/wiki/xacro">
     <link name="base_link">
       <visual>
@@ -16,15 +16,15 @@
       <inertial>
         <origin xyz="0.0 0 0"/>
-        <mass value="0.5"/>
-        <inertia ixx="0.01" ixy="0.0" ixz="0.0"
-                 iyy="0.01" iyz="0.0"
+        <mass value="10000"/>
+        <inertia ixx="0.0" ixy="0.0" ixz="0.0"
+                 iyy="0.0" iyz="0.0"
                  izz="0.03"/>
       </inertial>
     </link>
-    <gazebo reference="base_link">
+    <!--gazebo reference="base_link">
       <material>Gazebo/White</material>
-    </gazebo>
+    </gazebo-->
     <joint name="joint1_joint" type="revolute">
-      <origin xyz="0 0 0" rpy="0 0 1.57" />
+      <origin xyz="0 0 0" rpy="0 0 0" />
       <parent link="base_link"/>
       <child link="joint1_link" />
@@ -46,6 +46,6 @@
       </collision>
       <inertial>
-        <origin xyz="0.0 0 0"/>
-        <mass value="10"/>
+        <origin xyz="0 0 0"/>
+        <mass value="0.5"/>
         <inertia ixx="0.01" ixy="0.0" ixz="0.0"
                  iyy="0.01" iyz="0.0"
@@ -55,5 +55,5 @@
     <transmission name="trans_joint1_link">
       <type>transmission_interface/SimpleTransmission</type>
-      <joint name="joint1_link">
+      <joint name="joint1_joint">
         <hardwareInterface>hardware_interface/EffortJointInterface</hardwareInterface>
       </joint>
@@ -67,8 +67,8 @@
     </gazebo-->
     <joint name="joint2_joint" type="revolute">
-      <origin xyz="0 0 0" rpy="0 0 0"/>
+      <origin xyz="-0.05 0 0.48" rpy="0 0 0"/>
       <parent link="joint1_link"/>
       <child link="joint2_link" />
-      <axis xyz="0 0 1"/>
+      <axis xyz="1 0 0"/>
       <limit effort="1000.0" lower="-2.8" upper="2.8" velocity="0.5"/>
     </joint>
@@ -96,5 +96,5 @@
     <transmission name="trans_joint2_link">
       <type>transmission_interface/SimpleTransmission</type>
-      <joint name="joint2_link">
+      <joint name="joint2_joint">
         <hardwareInterface>hardware_interface/EffortJointInterface</hardwareInterface>
       </joint>
@@ -104,13 +104,13 @@
       </actuator>
     </transmission>
-    <gazebo reference="joint2_link">
+    <!--gazebo reference="joint2_link">
       <material>Gazebo/Grey</material>
-    </gazebo>
+    </gazebo-->
     <joint name="joint3_joint" type="revolute">
-      <origin xyz="0 0 0" rpy="0 0 0" />
+      <origin xyz="-0.07 -0.1 0" rpy="0 0 0" />
       <parent link="joint2_link"/>
       <child link="joint3_link" />
-      <axis xyz="0 0 1"/>
-      <limit effort="1000.0" lower="-3.14" upper="3.14" velocity="0.5"/>
+      <axis xyz="1 0 0"/>
+      <limit effort="1000.0" lower="-2.7" upper="2.7" velocity="0.5"/>
     </joint>
     <link name="joint3_link">
@@ -137,5 +137,5 @@
     <transmission name="trans_joint3_link">
       <type>transmission_interface/SimpleTransmission</type>
-      <joint name="joint3_link">
+      <joint name="joint3_joint">
         <hardwareInterface>hardware_interface/EffortJointInterface</hardwareInterface>
       </joint>
@@ -145,13 +145,13 @@
       </actuator>
     </transmission>
-    <gazebo reference="joint3_link">
+    <!--gazebo reference="joint3_link">
       <material>Gazebo/Grey</material>
-    </gazebo>
+    </gazebo-->
     <!-- Plugins -->
     <gazebo>
       <plugin name="gazebo_ros_control" filename="libgazebo_ros_control.so">
       </plugin>
-      <!--robotNamespace>/rms</robotNamespace>
-      <robotParam>/rms/robot_description</robotParam-->
+      <robotNamespace>/rms</robotNamespace>
+      <robotParam>/rms/robot_description</robotParam>
     </gazebo>
 </robot>
