Commit message: Scara0 working
Several files of scara0 have been changed. The robot an now spawn with correct PID value. A simple "wave" script has been added to test the joint;
Inverse kinematic equation should come.
PID for prismatic joint3, is not ideal

File: urdf/scara0.xacro (robot description, xacro)
@@ -1,4 +1,4 @@
 <?xml version="1.0" encoding="utf-8"?>
-<robot name="billy_v2" xmlns:xacro="http://www.ros.org/wiki/xacro">
+<robot name="scara0" xmlns:xacro="http://www.ros.org/wiki/xacro">
     <link name="base_link">
       <visual>
@@ -16,7 +16,7 @@
       <inertial>
         <origin xyz="0.0 0 0"/>
-        <mass value="0.5"/>
-        <inertia ixx="0.01" ixy="0.0" ixz="0.0"
-                 iyy="0.01" iyz="0.0"
+        <mass value="100"/>
+        <inertia ixx="0.0" ixy="0.0" ixz="0.0"
+                 iyy="0.0" iyz="0.0"
                  izz="0.03"/>
       </inertial>
@@ -47,5 +47,5 @@
       <inertial>
         <origin xyz="0.0 0 0"/>
-        <mass value="10"/>
+        <mass value="0.5"/>
         <inertia ixx="0.01" ixy="0.0" ixz="0.0"
                  iyy="0.01" iyz="0.0"
@@ -55,5 +55,5 @@
     <transmission name="trans_joint1_link">
       <type>transmission_interface/SimpleTransmission</type>
-      <joint name="joint1_link">
+      <joint name="joint1_joint">
         <hardwareInterface>hardware_interface/EffortJointInterface</hardwareInterface>
       </joint>
@@ -63,9 +63,9 @@
       </actuator>
     </transmission>
-    <!--gazebo reference="joint1_link">
+    <gazebo reference="joint1_link">
       <material>Gazebo/Grey</material>
-    </gazebo-->
+    </gazebo>
     <joint name="joint2_joint" type="revolute">
-      <origin xyz="0.1 0 0.12" rpy="0 0 0"/>
+      <origin xyz="0.11 0 0.12" rpy="0 0 0"/>
       <parent link="joint1_link"/>
       <child link="joint2_link" />
@@ -96,5 +96,5 @@
     <transmission name="trans_joint2_link">
       <type>transmission_interface/SimpleTransmission</type>
-      <joint name="joint2_link">
+      <joint name="joint2_joint">
         <hardwareInterface>hardware_interface/EffortJointInterface</hardwareInterface>
       </joint>
@@ -112,5 +112,5 @@
       <child link="joint3_link" />
       <axis xyz="0 0 1"/>
-      <limit effort="1000.0" lower="0" upper="0.06" velocity="0.5"/>
+      <limit effort="1000.0" lower="0" upper="0.06" velocity="0.01"/>
     </joint>
     <link name="joint3_link">
@@ -137,5 +137,5 @@
     <transmission name="trans_joint3_link">
       <type>transmission_interface/SimpleTransmission</type>
-      <joint name="joint3_link">
+      <joint name="joint3_joint">
         <hardwareInterface>hardware_interface/EffortJointInterface</hardwareInterface>
       </joint>
@@ -152,6 +152,6 @@
       <plugin name="gazebo_ros_control" filename="libgazebo_ros_control.so">
       </plugin>
-      <!--robotNamespace>/rms</robotNamespace>
-      <robotParam>/rms/robot_description</robotParam-->
+      <robotNamespace>/rms</robotNamespace>
+      <robotParam>/rms/robot_description</robotParam>
     </gazebo>
 </robot>

Commit message: Implementation of Inverse Kinematic for scara0
Added forward/inverse kinematic equation.
The good inverse kinematic function is inverse_kinematic2.
xy, quadrant and routine are demonstration of use of the robot
Only colors of the parts have been changes in .xacro file

File: urdf/scara0.xacro (robot description, xacro)
@@ -64,5 +64,5 @@
     </transmission>
     <gazebo reference="joint1_link">
-      <material>Gazebo/Grey</material>
+      <material>Gazebo/Yellow</material>
     </gazebo>
     <joint name="joint2_joint" type="revolute">
@@ -105,5 +105,5 @@
     </transmission>
     <gazebo reference="joint2_link">
-      <material>Gazebo/Grey</material>
+      <material>Gazebo/Orange</material>
     </gazebo>
     <joint name="joint3_joint" type="prismatic">
@@ -146,5 +146,5 @@
     </transmission>
     <gazebo reference="joint3_link">
-      <material>Gazebo/Grey</material>
+      <material>Gazebo/Red</material>
     </gazebo>
     <!-- Plugins -->

Commit message: Add gripper and camera
Add gripper stll and modifed xacro, lauch and yaml accordingly. The routine has been updated to do a pick and place movement. Some files of the gripper are missing (adding unnecessary complexity).
Add camera pluggin and position camera to see grabber. Rviz config saved.

File: urdf/scara0.xacro (robot description, xacro)
@@ -67,5 +67,5 @@
     </gazebo>
     <joint name="joint2_joint" type="revolute">
-      <origin xyz="0.11 0 0.12" rpy="0 0 0"/>
+      <origin xyz="0.11 0 0.27" rpy="0 0 0"/>
       <parent link="joint1_link"/>
       <child link="joint2_link" />
@@ -107,4 +107,30 @@
       <material>Gazebo/Orange</material>
     </gazebo>
+    <joint name="cam_joint" type="fixed">
+      <origin xyz="0.13 0 0.1" rpy="0 1.7 0" />
+      <parent link="joint2_link"/>
+      <child link="cam_link" />
+    </joint>
+    <link name="cam_link">
+      <!--visual>
+        <geometry>
+         <mesh scale="0.001 0.001 0.001" filename="package://rms_scara/meshes/scara0/scara0_joint2.stl"/>
+        </geometry>
+        <origin xyz="-0.1 0 -0.12" rpy="0 0 0"/>
+      </visual>
+      <collision>
+        <geometry>
+         <mesh scale="0.001 0.001 0.001" filename="package://rms_scara/meshes/scara0/scara0_joint2.stl"/>
+        </geometry>
+        <origin xyz="-0.1 0 -0.12" rpy="0 0 0"/>
+      </collision>
+      <inertial>
+        <origin xyz="0.0 0 0"/>
+        <mass value="0.5"/>
+        <inertia ixx="0.01" ixy="0.0" ixz="0.0"
+                 iyy="0.01" iyz="0.0"
+                 izz="0.03"/>
+      </inertial-->
+    </link>
     <joint name="joint3_joint" type="prismatic">
       <origin xyz="0.1 0 0.06" rpy="0 0 0" />
@@ -148,5 +174,117 @@
       <material>Gazebo/Red</material>
     </gazebo>
+    <joint name="gripper_main_joint" type="fixed">
+      <origin xyz="-0.03 0 -0.146" rpy="0 0 1.57" />
+      <parent link="joint3_link"/>
+      <child link="gripper_main_link" />
+    </joint>
+    <link name="gripper_main_link">
+      <visual>
+        <geometry>
+         <mesh scale="0.001 0.001 0.001" filename="package://rms_scara/meshes/scara0/scara0_gripper_main.stl"/>
+        </geometry>
+        <origin xyz="0 0 0" rpy="0 0 0"/>
+      </visual>
+      <collision>
+        <geometry>
+         <mesh scale="0.001 0.001 0.001" filename="package://rms_scara/meshes/scara0/scara0_gripper_main.stl"/>
+        </geometry>
+        <origin xyz="0 0 0" rpy="0 0 0"/>
+      </collision>
+      <inertial>
+        <origin xyz="0.0 0 0"/>
+        <mass value="0.5"/>
+        <inertia ixx="0.01" ixy="0.0" ixz="0.0"
+                 iyy="0.01" iyz="0.0"
+                 izz="0.03"/>
+      </inertial>
+    </link>
+    <gazebo reference="gripper_main_link">
+      <material>Gazebo/Red</material>
+    </gazebo>
+    <joint name="gripper_right_joint" type="prismatic">
+      <origin xyz="-0.01 0 0" rpy="0 0 0" />
+      <parent link="gripper_main_link"/>
+      <child link="gripper_right_link" />
+      <axis xyz="1 0 0"/>
+      <limit effort="1000.0" lower="0" upper="0.02" velocity="0.001"/>
+    </joint>
+    <link name="gripper_right_link">
+      <visual>
+        <geometry>
+         <mesh scale="0.001 0.001 0.001" filename="package://rms_scara/meshes/scara0/scara0_gripper_right.stl"/>
+        </geometry>
+        <origin xyz="0 0 0" rpy="0 0 0"/>
+      </visual>
+      <collision>
+        <geometry>
+         <mesh scale="0.001 0.001 0.001" filename="package://rms_scara/meshes/scara0/scara0_gripper_right.stl"/>
+        </geometry>
+        <origin xyz="0 0 0" rpy="0 0 0"/>
+      </collision>
+      <inertial>
+        <origin xyz="0.0 0 0"/>
+        <mass value="0.5"/>
+        <inertia ixx="0.01" ixy="0.0" ixz="0.0"
+                 iyy="0.01" iyz="0.0"
+                 izz="0.03"/>
+      </inertial>
+    </link>
+    <transmission name="trans_gripper_right_link">
+      <type>transmission_interface/SimpleTransmission</type>
+      <joint name="gripper_right_joint">
+        <hardwareInterface>hardware_interface/EffortJointInterface</hardwareInterface>
+      </joint>
+      <actuator name="ac_gripper_right_link">
+        <hardwareInterface>hardware_interface/EffortJointInterface</hardwareInterface>
+        <mechanicalReduction>1</mechanicalReduction>
+      </actuator>
+    </transmission>
+    <gazebo reference="gripper_right_link">
+      <material>Gazebo/Purple</material>
+    </gazebo>
+    <joint name="gripper_left_joint" type="prismatic">
+      <origin xyz="0.01 0 0" rpy="0 0 0" />
+      <parent link="gripper_main_link"/>
+      <child link="gripper_left_link" />
+      <axis xyz="1 0 0"/>
+      <limit effort="1000.0" lower="-0.02" upper="0" velocity="0.001"/>
+    </joint>
+    <link name="gripper_left_link">
+      <visual>
+        <geometry>
+         <mesh scale="0.001 0.001 0.001" filename="package://rms_scara/meshes/scara0/scara0_gripper_left.stl"/>
+        </geometry>
+        <origin xyz="0 0 0" rpy="0 0 0"/>
+      </visual>
+      <collision>
+        <geometry>
+         <mesh scale="0.001 0.001 0.001" filename="package://rms_scara/meshes/scara0/scara0_gripper_left.stl"/>
+        </geometry>
+        <origin xyz="0 0 0" rpy="0 0 0"/>
+      </collision>
+      <inertial>
+        <origin xyz="0.0 0 0"/>
+        <mass value="0.5"/>
+        <inertia ixx="0.01" ixy="0.0" ixz="0.0"
+                 iyy="0.01" iyz="0.0"
+                 izz="0.03"/>
+      </inertial>
+    </link>
+    <transmission name="trans_gripper_left_link">
+      <type>transmission_interface/SimpleTransmission</type>
+      <joint name="gripper_left_joint">
+        <hardwareInterface>hardware_interface/EffortJointInterface</hardwareInterface>
+      </joint>
+      <actuator name="ac_gripper_left_link">
+        <hardwareInterface>hardware_interface/EffortJointInterface</hardwareInterface>
+        <mechanicalReduction>1</mechanicalReduction>
+      </actuator>
+    </transmission>
+    <gazebo reference="gripper_left_link">
+      <material>Gazebo/Purple</material>
+    </gazebo>
     <!-- Plugins -->
+    <!--Control -->
     <gazebo>
       <plugin name="gazebo_ros_control" filename="libgazebo_ros_control.so">
@@ -155,3 +293,34 @@
       <robotParam>/rms/robot_description</robotParam>
     </gazebo>
+    <!-- Camera -->
+    <gazebo reference="cam_link"><sensor type="camera" name="myCam">
+      <update_rate>30.0</update_rate>
+      <camera name="head">
+        <horizontal_fov>1.04</horizontal_fov>
+        <image>
+          <width>720</width>
+          <height>480</height>
+          <format>R8G8B8</format>
+        </image>
+        <clip>
+          <near>0.1</near>
+          <far>50</far>
+        </clip>
+      </camera>
+      <plugin name="camera_controller" filename="libgazebo_ros_camera.so">
+        <alwaysOn>true</alwaysOn>
+        <updateRate>0</updateRate>
+        <cameraName>camera1</cameraName>
+        <imageTopicName>image_raw</imageTopicName>
+        <cameraInfoTopicName>camera_info</cameraInfoTopicName>
+        <frameName>camera</frameName>
+        <hackBaseline>0.07</hackBaseline>
+        <distortionK1>0.0</distortionK1>
+        <distortionK2>0.0</distortionK2>
+        <distortionK3>0.0</distortionK3>
+        <distortionT1>0.0</distortionT1>
+        <distortionT2>0.0</distortionT2>
+      </plugin>
+      </sensor>
+    </gazebo>
 </robot>

Commit message: Color recognision and world add
This commit is about color recognition.
Algorithm to detect color and align with pixels from the mask has been added.
Worlds and objects have been created to simulate different color of pen.

File: urdf/scara0.xacro (robot description, xacro)
@@ -26,5 +26,5 @@
     </gazebo>
     <joint name="joint1_joint" type="revolute">
-      <origin xyz="0 0 0" rpy="0 0 0" />
+      <origin xyz="0 0 0.01" rpy="0 0 0" />
       <parent link="base_link"/>
       <child link="joint1_link" />
@@ -67,5 +67,5 @@
     </gazebo>
     <joint name="joint2_joint" type="revolute">
-      <origin xyz="0.11 0 0.27" rpy="0 0 0"/>
+      <origin xyz="0.2 0 0.147" rpy="0 0 0"/>
       <parent link="joint1_link"/>
       <child link="joint2_link" />
@@ -78,5 +78,5 @@
          <mesh scale="0.001 0.001 0.001" filename="package://rms_scara/meshes/scara0/scara0_joint2.stl"/>
         </geometry>
-        <origin xyz="-0.1 0 -0.12" rpy="0 0 0"/>
+        <origin xyz="0 0 0" rpy="0 0 0"/>
       </visual>
       <collision>
@@ -84,5 +84,5 @@
          <mesh scale="0.001 0.001 0.001" filename="package://rms_scara/meshes/scara0/scara0_joint2.stl"/>
         </geometry>
-        <origin xyz="-0.1 0 -0.12" rpy="0 0 0"/>
+        <origin xyz="0 0 0" rpy="0 0 0"/>
       </collision>
       <inertial>
@@ -108,5 +108,5 @@
     </gazebo>
     <joint name="cam_joint" type="fixed">
-      <origin xyz="0.13 0 0.1" rpy="0 1.7 0" />
+      <origin xyz="0.3 0 0.1" rpy="0 2.0 0" />
       <parent link="joint2_link"/>
       <child link="cam_link" />
@@ -134,9 +134,9 @@
     </link>
     <joint name="joint3_joint" type="prismatic">
-      <origin xyz="0.1 0 0.06" rpy="0 0 0" />
+      <origin xyz="0.2 0 0.1" rpy="0 0 0" />
       <parent link="joint2_link"/>
       <child link="joint3_link" />
       <axis xyz="0 0 1"/>
-      <limit effort="1000.0" lower="0" upper="0.06" velocity="0.01"/>
+      <limit effort="1000.0" lower="0" upper="0.1" velocity="0.01"/>
     </joint>
     <link name="joint3_link">
@@ -145,5 +145,5 @@
          <mesh scale="0.001 0.001 0.001" filename="package://rms_scara/meshes/scara0/scara0_joint3.stl"/>
         </geometry>
-        <origin xyz="-0.20 0 -0.18" rpy="0 0 0"/>
+        <origin xyz="0 0 0" rpy="0 0 0"/>
       </visual>
       <collision>
@@ -151,5 +151,5 @@
          <mesh scale="0.001 0.001 0.001" filename="package://rms_scara/meshes/scara0/scara0_joint3.stl"/>
         </geometry>
-        <origin xyz="-0.20 0 -0.18" rpy="0 0 0"/>
+        <origin xyz="0 0 0" rpy="0 0 0"/>
       </collision>
       <inertial>
@@ -175,5 +175,5 @@
     </gazebo>
     <joint name="gripper_main_joint" type="fixed">
-      <origin xyz="-0.03 0 -0.146" rpy="0 0 1.57" />
+      <origin xyz="-0.025 0 -0.205" rpy="0 0 1.57" />
       <parent link="joint3_link"/>
       <child link="gripper_main_link" />
