Commit message: rms_scara2 working demonstration
rms_scara2 is now working and a demonstration is available in scara2_wave.py.
Next step would be to add a new joint on the gripper_main to calibrate the orientation.
Next next step, would be the improve the calibration model with an holomonic matrix

File: urdf/scara2.xacro (robot description, xacro)
@@ -10,5 +10,5 @@
       </visual>
       <collision>
-        <origin xyz="0 0 0" rpy="0 0 0"/>
+        <origin xyz="0 0 0" rpy="1.5707 0 3.1416"/>
         <geometry>
           <mesh scale="0.010 0.010 0.010" filename="package://rms_scara/meshes/scara2/scara2_base_link.stl"/>
@@ -28,5 +28,5 @@
     <!-- ____________________ Shafts and screw ____________________ -->
     <joint name="shaft1_joint" type="fixed">
-      <origin xyz="0.016 0.01 0.028" rpy="0 0 0" />
+      <origin xyz="0.0175 0.005 0.0303" rpy="0 0 0" />
       <parent link="joint2_link"/>
       <child link="shaft1_link" />
@@ -54,5 +54,5 @@
     </link>
     <joint name="shaft2_joint" type="fixed">
-      <origin xyz="-0.035 0.01 0" rpy="0 0 0" />
+      <origin xyz="-0.035 0.005 0" rpy="0 0 0" />
       <parent link="joint2_link"/>
       <child link="shaft2_link" />
@@ -80,5 +80,5 @@
     </link>
     <joint name="shaft3_joint" type="fixed">
-      <origin xyz="0.016 0.01 -0.028" rpy="0 0 0" />
+      <origin xyz="0.0175 0.01 -0.0303" rpy="0 0 0" />
       <parent link="joint2_link"/>
       <child link="shaft3_link" />
@@ -105,4 +105,5 @@
       </inertial>
     </link>
+    <!--
     <joint name="screw_joint" type="fixed">
       <origin xyz="0.045 0 0" rpy="0 0 0" />
@@ -131,7 +132,8 @@
       </inertial>
     </link>
+    -->
     <!-- ____________________ Hat ____________________ -->
     <joint name="top_joint" type="fixed">
-      <origin xyz="0 0.4 0" rpy="0 2.09 0" />
+      <origin xyz="0 0.41 0" rpy="0 3.141 3.14" />
       <parent link="joint2_link"/>
       <child link="top_link" />
@@ -160,9 +162,9 @@
     <!-- ____________________ Joints ____________________ -->
     <joint name="joint1_joint" type="prismatic">
-      <origin xyz="0 0.035 0" rpy="0 0 0" />
+      <origin xyz="0 0.115 0" rpy="0 0.523 0" />
       <parent link="joint2_link"/>
       <child link="joint1_link" />
       <axis xyz="0 1 0"/>
-      <limit effort="1000.0" lower="0" upper="1" velocity="0.5"/>
+      <limit effort="1000.0" lower="0.0" upper="0.26" velocity="0.2"/>
     </joint>
     <link name="joint1_link">
@@ -205,5 +207,5 @@
       <child link="joint2_link" />
       <axis xyz="0 1 0"/>
-      <limit effort="1000.0" lower="-2.80" upper="2.80" velocity="0.5"/>
+      <limit effort="1000.0" lower="-2.80" upper="2.80" velocity="0.2"/>
     </joint>
     <link name="joint2_link">
@@ -241,36 +243,10 @@
       <material>Gazebo/Orange</material>
     </gazebo>
-    <joint name="cam_joint" type="fixed">
-      <origin xyz="0 0 0" rpy="0 0 0" />
-      <parent link="joint2_link"/>
-      <child link="cam_link" />
-    </joint>
-    <link name="cam_link">
-      <!--visual>
-        <geometry>
-         <mesh scale="0.001 0.001 0.001" filename="package://rms_scara/meshes/scara2/scara2_joint2.stl"/>
-        </geometry>
-        <origin xyz="-0.1 0 -0.12" rpy="0 0 0"/>
-      </visual>
-      <collision>
-        <geometry>
-         <mesh scale="0.001 0.001 0.001" filename="package://rms_scara/meshes/scara2/scara2_joint2.stl"/>
-        </geometry>
-        <origin xyz="-0.1 0 -0.12" rpy="0 0 0"/>
-      </collision>
-      <inertial>
-        <origin xyz="0.0 0 0"/>
-        <mass value="0.5"/>
-        <inertia ixx="0.01" ixy="0.0" ixz="0.0"
-                 iyy="0.01" iyz="0.0"
-                 izz="0.03"/>
-      </inertial-->
-    </link>
     <joint name="joint3_joint" type="revolute">
-      <origin xyz="0 -0.035 -0.15" rpy="0 0 0" />
+      <origin xyz="0 -0.035 -0.15" rpy="3.14 3.14 0" />
       <parent link="joint1_link"/>
       <child link="joint3_link" />
       <axis xyz="0 1 0"/>
-      <limit effort="1000.0" lower="-2.8" upper="2.8" velocity="0.5"/>
+      <limit effort="1000.0" lower="-2.8" upper="2.8" velocity="0.1"/>
     </joint>
     <link name="joint3_link">
@@ -308,7 +284,7 @@
       <material>Gazebo/Red</material>
     </gazebo>
-    <!--
+    <!-- ____________________ Gripper ____________________ -->
     <joint name="gripper_main_joint" type="fixed">
-      <origin xyz="-0.025 0 -0.205" rpy="0 0 1.57" />
+      <origin xyz="0 0.070 -0.12" rpy="-1.57 3.14 3.14" />
       <parent link="joint3_link"/>
       <child link="gripper_main_link" />
@@ -339,20 +315,20 @@
     </gazebo>
     <joint name="gripper_right_joint" type="prismatic">
-      <origin xyz="-0.01 0 0" rpy="0 0 0" />
+      <origin xyz="0.0078 -0.01 -0.05" rpy="1.57 0 0" />
       <parent link="gripper_main_link"/>
       <child link="gripper_right_link" />
       <axis xyz="1 0 0"/>
-      <limit effort="1000.0" lower="0" upper="0.02" velocity="0.001"/>
+      <limit effort="1000.0" lower="0" upper="0.025" velocity="0.1"/>
     </joint>
     <link name="gripper_right_link">
       <visual>
         <geometry>
-         <mesh scale="0.001 0.001 0.001" filename="package://rms_scara/meshes/scara2/scara2_gripper_right.stl"/>
-        </geometry>
-        <origin xyz="0 0 0" rpy="0 0 0"/>
-      </visual>
-      <collision>
-        <geometry>
-         <mesh scale="0.001 0.001 0.001" filename="package://rms_scara/meshes/scara2/scara2_gripper_right.stl"/>
+         <mesh scale="0.001 0.001 0.001" filename="package://rms_scara/meshes/scara2/scara2_gripper_right_2.stl"/>
+        </geometry>
+        <origin xyz="0 0 0" rpy="0 0 0"/>
+      </visual>
+      <collision>
+        <geometry>
+         <mesh scale="0.001 0.001 0.001" filename="package://rms_scara/meshes/scara2/scara2_gripper_right_2.stl"/>
         </geometry>
         <origin xyz="0 0 0" rpy="0 0 0"/>
@@ -380,20 +356,20 @@
     </gazebo>
     <joint name="gripper_left_joint" type="prismatic">
-      <origin xyz="0.01 0 0" rpy="0 0 0" />
+      <origin xyz="-0.0078 -0.05 -0.05" rpy="1.57 0 3.14" />
       <parent link="gripper_main_link"/>
       <child link="gripper_left_link" />
       <axis xyz="1 0 0"/>
-      <limit effort="1000.0" lower="-0.02" upper="0" velocity="0.001"/>
+      <limit effort="1000.0" lower="0" upper="0.025" velocity="0.1"/>
     </joint>
     <link name="gripper_left_link">
       <visual>
         <geometry>
-         <mesh scale="0.001 0.001 0.001" filename="package://rms_scara/meshes/scara2/scara2_gripper_left.stl"/>
-        </geometry>
-        <origin xyz="0 0 0" rpy="0 0 0"/>
-      </visual>
-      <collision>
-        <geometry>
-         <mesh scale="0.001 0.001 0.001" filename="package://rms_scara/meshes/scara2/scara2_gripper_left.stl"/>
+         <mesh scale="0.001 0.001 0.001" filename="package://rms_scara/meshes/scara2/scara2_gripper_left_2.stl"/>
+        </geometry>
+        <origin xyz="0 0 0" rpy="0 0 0"/>
+      </visual>
+      <collision>
+        <geometry>
+         <mesh scale="0.001 0.001 0.001" filename="package://rms_scara/meshes/scara2/scara2_gripper_left_2.stl"/>
         </geometry>
         <origin xyz="0 0 0" rpy="0 0 0"/>
@@ -420,7 +396,34 @@
       <material>Gazebo/Purple</material>
     </gazebo>
-    -->
-    <!-- Plugins -->
-    <!--Control -->
+    <!-- ____________________ Camera ____________________ -->
+    <joint name="cam_joint" type="fixed">
+      <origin xyz="0 -0.12 0.15" rpy="0 2.0 -1.57"/>
+      <parent link="gripper_main_link"/>
+      <child link="cam_link" />
+    </joint>
+    <link name="cam_link">
+      <!--
+      <visual>
+        <geometry>
+          <cylinder length="0.01" radius="0.01"/>
+        </geometry>
+        <origin xyz="0 0 0" rpy="0 0 0"/>
+      </visual>
+      <collision>
+        <geometry>
+          <cylinder length="0.1" radius="0.1"/>
+        </geometry>
+        <origin xyz="0 0 0" rpy="0 0 0"/>
+      </collision>
+      <inertial>
+        <origin xyz="0.0 0 0"/>
+        <mass value="0.5"/>
+        <inertia ixx="0.01" ixy="0.0" ixz="0.0"
+                 iyy="0.01" iyz="0.0"
+                 izz="0.03"/>
+      </inertial>
+      -->
+    </link>
+    <!-- ____________________ Plugins ____________________ -->
     <gazebo>
       <plugin name="gazebo_ros_control" filename="libgazebo_ros_control.so">
@@ -430,5 +433,4 @@
     </gazebo>
     <!-- Camera -->
-    <!--
     <gazebo reference="cam_link"><sensor type="camera" name="myCam">
       <update_rate>30.0</update_rate>
@@ -461,4 +463,3 @@
       </sensor>
     </gazebo>
-    -->
 </robot>

Commit message: Add a joint on the gripper_main
This new joint allows rotation on the gripper_main. This allows to grab a pen in any orientation as long as your on top of it.
The URDF part has been updated and the camera position has well. Tests have been made and assessed.
Camera could be better though.

File: urdf/scara2.xacro (robot description, xacro)
@@ -285,8 +285,10 @@
     </gazebo>
     <!-- ____________________ Gripper ____________________ -->
-    <joint name="gripper_main_joint" type="fixed">
+    <joint name="gripper_main_joint" type="revolute">
       <origin xyz="0 0.070 -0.12" rpy="-1.57 3.14 3.14" />
       <parent link="joint3_link"/>
       <child link="gripper_main_link" />
+      <axis xyz="0 0 1"/>
+      <limit effort="1000.0" lower="-3.14" upper="3.14" velocity="0.1"/>
     </joint>
     <link name="gripper_main_link">
@@ -295,5 +297,5 @@
          <mesh scale="0.001 0.001 0.001" filename="package://rms_scara/meshes/scara2/scara2_gripper_main.stl"/>
         </geometry>
-        <origin xyz="0 0 0" rpy="0 0 0"/>
+        <origin xyz="0 0.030 0" rpy="0 0 0"/>
       </visual>
       <collision>
@@ -301,19 +303,29 @@
          <mesh scale="0.001 0.001 0.001" filename="package://rms_scara/meshes/scara2/scara2_gripper_main.stl"/>
         </geometry>
-        <origin xyz="0 0 0" rpy="0 0 0"/>
-      </collision>
-      <inertial>
-        <origin xyz="0.0 0 0"/>
-        <mass value="0.5"/>
-        <inertia ixx="0.01" ixy="0.0" ixz="0.0"
-                 iyy="0.01" iyz="0.0"
-                 izz="0.03"/>
-      </inertial>
-    </link>
+        <origin xyz="0 0.030 0" rpy="0 0 0"/>
+      </collision>
+      <inertial>
+        <origin xyz="0.0 0 0"/>
+        <mass value="0.5"/>
+        <inertia ixx="0.01" ixy="0.0" ixz="0.0"
+                 iyy="0.01" iyz="0.0"
+                 izz="0.03"/>
+      </inertial>
+    </link>
+    <transmission name="trans_gripper_main_link">
+      <type>transmission_interface/SimpleTransmission</type>
+      <joint name="gripper_main_joint">
+        <hardwareInterface>hardware_interface/EffortJointInterface</hardwareInterface>
+      </joint>
+      <actuator name="ac_gripper_main_link">
+        <hardwareInterface>hardware_interface/EffortJointInterface</hardwareInterface>
+        <mechanicalReduction>1</mechanicalReduction>
+      </actuator>
+    </transmission>
     <gazebo reference="gripper_main_link">
       <material>Gazebo/Red</material>
     </gazebo>
     <joint name="gripper_right_joint" type="prismatic">
-      <origin xyz="0.0078 -0.01 -0.05" rpy="1.57 0 0" />
+      <origin xyz="0.0078 0.018 -0.05" rpy="1.57 0 0" />
       <parent link="gripper_main_link"/>
       <child link="gripper_right_link" />
@@ -356,5 +368,5 @@
     </gazebo>
     <joint name="gripper_left_joint" type="prismatic">
-      <origin xyz="-0.0078 -0.05 -0.05" rpy="1.57 0 3.14" />
+      <origin xyz="-0.0078 -0.022 -0.05" rpy="1.57 0 3.14" />
       <parent link="gripper_main_link"/>
       <child link="gripper_left_link" />
@@ -398,6 +410,6 @@
     <!-- ____________________ Camera ____________________ -->
     <joint name="cam_joint" type="fixed">
-      <origin xyz="0 -0.12 0.15" rpy="0 2.0 -1.57"/>
-      <parent link="gripper_main_link"/>
+      <origin xyz="0 -0.05 -0.22" rpy="0 -0.5 1.57"/>
+      <parent link="joint3_link"/>
       <child link="cam_link" />
     </joint>
